File: board/board.kicad_pcb (KiCad board)
At the start: 2 copper layers, 21 x 13 mm, 1 part

Commit message: initial
Parts:
- removed LOGO1: Logo_Open_Hardware_Small, Symbol:OSHW-Symbol_6.7x6mm_SilkScreen
- added C1: 10pF, Capacitor_SMD:C_0603_1608Metric, B.Cu at (87.0, 72.6)
- added C2: 1uF, Capacitor_SMD:C_0603_1608Metric, B.Cu at (92.7, 73.3)
- added C3: 10pF, Capacitor_SMD:C_0603_1608Metric, B.Cu at (87.0, 74.2)
- added C4: 1uF, Capacitor_SMD:C_0603_1608Metric, B.Cu at (91.1, 73.3)
- added C5: 1uF, Capacitor_SMD:C_0603_1608Metric, B.Cu at (92.8, 62.4)
- added C6: 1uF, Capacitor_SMD:C_0603_1608Metric, B.Cu at (87.4, 62.9)
- added C7: 10uF, Capacitor_SMD:C_0603_1608Metric, B.Cu at (87.4, 64.5)
- added FB1: Ferrite_Bead_Small, Inductor_SMD:L_0603_1608Metric, B.Cu at (94.3, 73.3)
- added J1: 002_SPI_2x5, on_edge:on_edge_2x05_device, F.Cu at (85.0, 51.5)
- added J3: 007_ADC_2x5, on_edge:on_edge_2x05_host, F.Cu at (106.0, 51.5)
- added J4: 007_ADC_2x5, on_edge:on_edge_2x05_host, F.Cu at (106.0, 67.5)
- added J5: 007_ADC_2x5, on_edge:on_edge_2x05_host, F.Cu at (106.0, 83.5)
- added J6: 007_ADC_2x5, on_edge:on_edge_2x05_host, F.Cu at (106.0, 99.5)
- added R1: 10k, Resistor_SMD:R_0603_1608Metric, B.Cu at (89.5, 73.3)
- added U1: ADS131M08, Package_DFN_QFN:WQFN-32-1EP_5x5mm_P0.5mm_EP3.1x3.1mm, B.Cu at (94.6, 67.7)
- added Y1: 8MhZ, Crystal:Crystal_SMD_5032-2Pin_5.0x3.2mm, B.Cu at (87.1, 68.6)
Routing:
- net GND: track 0.00 -> 128.3 mm, vias 0 -> 6
- net +3.3V: track 0.00 -> 106.4 mm, vias 0 -> 11
- net +5V: track 0.00 -> 93.0 mm, vias 0 -> 7
- net /adc/AIN_7P: track 0.00 -> 39.7 mm, vias 0 -> 1
- net /adc/AIN_6N: track 0.00 -> 36.9 mm, vias 0 -> 1
- net /adc/~{CS}: track 0.00 -> 35.6 mm, vias 0 -> 2
- net /adc/~{RESET}: track 0.00 -> 34.7 mm, vias 0 -> 2
- net /adc/AIN_6P: track 0.00 -> 33.6 mm, vias 0 -> 1
- net /adc/AIN_7N: track 0.00 -> 32.8 mm, vias 0 -> 2
- net /adc/AIN_1N: track 0.00 -> 22.8 mm
- net /adc/AIN_5P: track 0.00 -> 22.4 mm, vias 0 -> 1
- net /adc/SCLK: track 0.00 -> 22.4 mm, vias 0 -> 1
- net /adc/SDI: track 0.00 -> 21.8 mm, vias 0 -> 1
- net /adc/SDO: track 0.00 -> 21.8 mm, vias 0 -> 1
- net /adc/~{DRDY}: track 0.00 -> 21.0 mm, vias 0 -> 1
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Other:
- board size 21 x 13 mm -> 21 x 61 mm
- rule pad_to_mask_clearance: 0 -> 0.051
- board text added: "osf.002.v0.2"
- board text added: "osf.007.v0.2"
- board text added: "osf.b056.v0.1"
